Commit message: added wire chain to urdf

File: resources/m900ib400l/m900ib400l_spherized.urdf (robot description, URDF)
Before this commit: robot spherized, 7 links, 6 joints
Links:
- link link_3: geometry collision sphere radius=0.19399; collision sphere radius=0.242005

Commit message: added way to explicitly add endeffector collisions in the robots json

File: resources/m900ib400l/m900ib400l_spherized.urdf (robot description, URDF)
Before this commit: robot spherized, 7 links, 6 joints
Links:
- link link_3: geometry collision sphere radius=0.182005; collision sphere radius=0.19399
- link link_6: geometry collision sphere radius=0.07; collision sphere radius=0.07

Commit message: update m900

File: resources/m900ib400l/m900ib400l_spherized.urdf (robot description, URDF)
Before this commit: robot spherized, 7 links, 6 joints
Links:
- link link_3: geometry collision sphere radius=0.162005; collision sphere radius=0.16713
